File: aula02/aula2-projeto.brd (EAGLE design)
At the start: 257.9 x 59.7 mm, 11 parts, among them U1 ARDUINO-UNO-R3-SHIELD

Commit message: refactor: .ino code
Parts:
- R1, R2, R3: value 1.5k -> 150
Connections:
- new net U1_5V: S1.1, S1.2, S2.1, S2.2, U1.5V
- new net U1_D3: R1.1, U1.D3
- net U1_GND: no longer S1.1, S1.2, S2.1, S2.2
Changed lines of the file:
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@@
 </autorouter>
 <elements>
-<element name="R1" library="Tinkercad" library_urn="urn:adsk.eagle:library:30890021" package="RESAD1016W63L850D250B" package3d_urn="urn:adsk.eagle:package:31513020/2" value="1.5k" x="223.5364" y="41.3266" rot="R180" smashed="yes"/>
+<element name="R1" library="Tinkercad" library_urn="urn:adsk.eagle:library:30890021" package="RESAD1016W63L850D250B" package3d_urn="urn:adsk.eagle:package:31513020/2" value="150" x="223.5364" y="41.3266" rot="R180" smashed="yes"/>
 <element name="D2" library="Tinkercad" library_urn="urn:adsk.eagle:library:30890021" package="LEDRD254W60D565H860B_W" package3d_urn="urn:adsk.eagle:package:16378509/3" value="WHITE" x="217.1864" y="43.8666" rot="R180" smashed="yes">
 <attribute name="CATEGORY" value="Opto-Electronic" x="217.1864" y="43.8666" size="1.778" layer="27" display="off"/>
@@
 <attribute name="VALUE" value="LED_BLUE" x="191.7864" y="43.8666" size="1.778" layer="27" display="off"/>
 </element>
-<element name="R2" library="Tinkercad" library_urn="urn:adsk.eagle:library:30890021" package="RESAD1016W63L850D250B" package3d_urn="urn:adsk.eagle:package:31513020/2" value="1.5k" x="198.1364" y="41.3266" rot="R180" smashed="yes"/>
+<element name="R2" library="Tinkercad" library_urn="urn:adsk.eagle:library:30890021" package="RESAD1016W63L850D250B" package3d_urn="urn:adsk.eagle:package:31513020/2" value="150" x="198.1364" y="41.3266" rot="R180" smashed="yes"/>
 <element name="D1" library="Tinkercad" library_urn="urn:adsk.eagle:library:30890021" package="LEDRD254W60D565H860B" package3d_urn="urn:adsk.eagle:package:16378508/2" value="RED" x="242.5864" y="43.8666" rot="R180" smashed="yes">
 <attribute name="CATEGORY" value="Opto-Electronic" x="242.5864" y="43.8666" size="1.778" layer="27" display="off"/>
@@
 <attribute name="VALUE" value="LED_RED" x="242.5864" y="43.8666" size="1.778" layer="27" display="off"/>
 </element>
-<element name="R3" library="Tinkercad" library_urn="urn:adsk.eagle:library:30890021" package="RESAD1016W63L850D250B" package3d_urn="urn:adsk.eagle:package:31513020/2" value="1.5k" x="248.9364" y="41.3266" rot="R180" smashed="yes"/>
+<element name="R3" library="Tinkercad" library_urn="urn:adsk.eagle:library:30890021" package="RESAD1016W63L850D250B" package3d_urn="urn:adsk.eagle:package:31513020/2" value="150" x="248.9364" y="41.3266" rot="R180" smashed="yes"/>
 <element name="U1" library="Tinkercad" library_urn="urn:adsk.eagle:library:30890021" package="ARDUINO-UNO-R3-SHIELD" package3d_urn="urn:adsk.eagle:package:32092383/4" value="ARDUINO-UNO-R3-SHIELD" x="47.885" y="29.845" rot="R270" smashed="yes"/>
+<element name="R6" library="Tinkercad" library_urn="urn:adsk.eagle:library:30890021" package="RESAD1016W63L850D250B" package3d_urn="urn:adsk.eagle:package:31513020/2" value="10k" x="121.9364" y="13.3866" rot="R90" smashed="yes"/>
 <element name="R4" library="Tinkercad" library_urn="urn:adsk.eagle:library:30890021" package="RESAD1016W63L850D250B" package3d_urn="urn:adsk.eagle:package:31513020/2" value="10k" x="139.7164" y="13.3866" rot="R90" smashed="yes"/>
 <element name="S2" library="Tinkercad" library_urn="urn:adsk.eagle:library:30890021" package="SWITCH-MOMENTARY-PTH-6.5MM" package3d_urn="urn:adsk.eagle:package:32246662/3" value="SWITCH_MOMENTARY" x="137.1764" y="29.8966" rot="R90" smashed="yes"/>
-<element name="R6" library="Tinkercad" library_urn="urn:adsk.eagle:library:30890021" package="RESAD1016W63L850D250B" package3d_urn="urn:adsk.eagle:package:31513020/2" value="10k" x="121.9364" y="13.3866" rot="R90" smashed="yes"/>
 <element name="S1" library="Tinkercad" library_urn="urn:adsk.eagle:library:30890021" package="SWITCH-MOMENTARY-PTH-6.5MM" package3d_urn="urn:adsk.eagle:package:32246662/3" value="SWITCH_MOMENTARY" x="119.3964" y="29.8966" rot="R90" smashed="yes"/>
 </elements>
@@
 <wire x1="218.4564" y1="43.8666" x2="218.4564" y2="41.3266" width="0" layer="19" extent="1-1"/>
 </signal>
+<signal name="U1_D3">
+<contactref element="R1" pad="1"/>
+<contactref element="U1" pad="D3"/>
+<wire x1="228.6164" y1="41.3266" x2="65.665" y2="53.975" width="0" layer="19" extent="1-1"/>
+</signal>
 <signal name="U1_GND">
 <contactref element="D1" pad="2"/>
-<contactref element="D2" pad="2"/>
-<contactref element="D3" pad="2"/>
 <contactref element="U1" pad="GND@0"/>
 <contactref element="U1" pad="GND@1"/>
@@
 <contactref element="R6" pad="1"/>
 <contactref element="R4" pad="1"/>
-<contactref element="S1" pad="1"/>
-<contactref element="S2" pad="1"/>
-<contactref element="S1" pad="2"/>
-<contactref element="S2" pad="2"/>
+<contactref element="D3" pad="2"/>
+<contactref element="D2" pad="2"/>
 <wire x1="50.425" y1="5.715" x2="52.965" y2="5.715" width="0" layer="19" extent="1-1"/>
 <wire x1="50.425" y1="5.715" x2="36.455" y2="53.975" width="0" layer="19" extent="1-1"/>
-<wire x1="52.965" y1="5.715" x2="117.1358" y2="26.6454" width="0" layer="19" extent="1-1"/>
-<wire x1="117.1358" y1="26.6454" x2="117.1358" y2="33.1478" width="0" layer="19" extent="1-1"/>
-<wire x1="117.1358" y1="26.6454" x2="134.9158" y2="26.6454" width="0" layer="19" extent="1-1"/>
-<wire x1="134.9158" y1="26.6454" x2="134.9158" y2="33.1478" width="0" layer="19" extent="1-1"/>
-<wire x1="121.9364" y1="8.3066" x2="117.1358" y2="26.6454" width="0" layer="19" extent="1-1"/>
+<wire x1="52.965" y1="5.715" x2="121.9364" y2="8.3066" width="0" layer="19" extent="1-1"/>
 <wire x1="121.9364" y1="8.3066" x2="139.7164" y2="8.3066" width="0" layer="19" extent="1-1"/>
-<wire x1="190.5164" y1="43.8666" x2="134.9158" y2="33.1478" width="0" layer="19" extent="1-1"/>
-<wire x1="215.9164" y1="43.8666" x2="190.5164" y2="43.8666" width="0" layer="19" extent="1-1"/>
+<wire x1="139.7164" y1="8.3066" x2="190.5164" y2="43.8666" width="0" layer="19" extent="1-1"/>
+<wire x1="190.5164" y1="43.8666" x2="215.9164" y2="43.8666" width="0" layer="19" extent="1-1"/>
 <wire x1="241.3164" y1="43.8666" x2="215.9164" y2="43.8666" width="0" layer="19" extent="1-1"/>
 </signal>
@@
 <contactref element="R6" pad="2"/>
 <contactref element="S1" pad="3"/>
+<contactref element="U1" pad="D8"/>
 <contactref element="S1" pad="4"/>
-<contactref element="U1" pad="D8"/>
 <wire x1="121.657" y1="26.6454" x2="121.657" y2="33.1478" width="0" layer="19" extent="1-1"/>
 <wire x1="121.9364" y1="18.4666" x2="121.657" y2="26.6454" width="0" layer="19" extent="1-1"/>
-<wire x1="121.657" y1="33.1478" x2="51.695" y2="53.975" width="0" layer="19" extent="1-1"/>
+<wire x1="51.695" y1="53.975" x2="121.657" y2="33.1478" width="0" layer="19" extent="1-1"/>
+</signal>
+<signal name="U1_5V">
+<contactref element="S2" pad="2"/>
+<contactref element="S2" pad="1"/>
+<contactref element="U1" pad="5V"/>
+<contactref element="S1" pad="1"/>
+<contactref element="S1" pad="2"/>
+<wire x1="134.9158" y1="33.1478" x2="134.9158" y2="26.6454" width="0" layer="19" extent="1-1"/>
+<wire x1="134.9158" y1="33.1478" x2="117.1358" y2="33.1478" width="0" layer="19" extent="1-1"/>
+<wire x1="117.1358" y1="26.6454" x2="117.1358" y2="33.1478" width="0" layer="19" extent="1-1"/>
+<wire x1="47.885" y1="5.715" x2="117.1358" y2="26.6454" width="0" layer="19" extent="1-1"/>
 </signal>
 </signals>
